File: hardware/schematic/blink1_v2d.brd (EAGLE design)
At the start: 14.9 x 11.2 mm, 12 parts, among them P1 TPTP11SQ, U1 PIC16F1455ML, X1 USB

Commit message: more modest changes to blink1mk2 v2d idea
Parts:
- added IN: TPSQTP12SQ, testpad:TP12SQ
- renumbered TP1 to GND, TP2 to +5V, TP3 to DAT
Connections:
- new net N$2: U1.1
- new net N$3: U1.6
- new net N$4: U1.5
- new net N$5: U1.2
- new net N$6: U1.4
- net PGC: now also IN.TP
Routing:
- net PGC: track 0.00 -> 7.72 mm, vias 0 -> 1
Other:
- board text added: "blink1_v2d"
- board text removed: "+5"
- board text removed: "DO"
- board text removed: "Gnd"
- board text removed: "blink1_v2c5"
