File: hardware/schematic/blink1_v2d.sch (EAGLE design)
At the start: 12 parts, among them P1 TPTP11SQ, U1 PIC16F1455ML, X1 USB

Commit message: more modest changes to blink1mk2 v2d idea
Parts:
- removed TP1, TP3: TPSQTP12SQ, testpad:TPSQTP12SQ
- added DAT, GND, IN: TPSQTP12SQ, testpad:TPSQTP12SQ
- renumbered TP2 to +5V
Connections:
- new net N$2: U1.RA5
- new net N$3: U1.RC3
- new net N$4: U1.RC4
- new net N$5: U1.RA4
- new net N$6: U1.RC5
- net DO: now also DAT.TP; no longer TP3.TP
- net GND: now also GND.TP; no longer TP1.TP
- net PGC: now also IN.TP
Other:
- moved on the sheet: C3
Changed lines of the file:
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@@
 <part name="P+7" library="supply1" deviceset="+5V" device=""/>
 <part name="GND3" library="SparkFun-20110517" deviceset="GND" device=""/>
-<part name="TP1" library="testpad" deviceset="TPSQ" device="TP12SQ" value="TPSQTP12SQ"/>
-<part name="TP2" library="testpad" deviceset="TPSQ" device="TP12SQ" value="TPSQTP12SQ"/>
-<part name="TP3" library="testpad" deviceset="TPSQ" device="TP12SQ" value="TPSQTP12SQ"/>
+<part name="GND" library="testpad" deviceset="TPSQ" device="TP12SQ" value="TPSQTP12SQ"/>
+<part name="+5V" library="testpad" deviceset="TPSQ" device="TP12SQ" value="TPSQTP12SQ"/>
+<part name="DAT" library="testpad" deviceset="TPSQ" device="TP12SQ" value="TPSQTP12SQ"/>
+<part name="IN" library="testpad" deviceset="TPSQ" device="TP12SQ" value="TPSQTP12SQ"/>
 </parts>
 <sheets>
@@
 </instance>
 <instance part="GND8" gate="1" x="137.16" y="165.1"/>
-<instance part="GND11" gate="1" x="208.28" y="86.36"/>
+<instance part="GND11" gate="1" x="220.98" y="86.36"/>
 <instance part="P+1" gate="1" x="116.84" y="187.96" smashed="yes">
 <attribute name="VALUE" x="119.38" y="190.5" size="1.778" layer="96" rot="R180"/>
@@
 <instance part="U1" gate="G$1" x="165.1" y="96.52"/>
 <instance part="C2" gate="G$1" x="137.16" y="175.26"/>
-<instance part="C3" gate="G$1" x="208.28" y="93.98"/>
+<instance part="C3" gate="G$1" x="220.98" y="93.98"/>
 <instance part="P1" gate="G$1" x="86.36" y="111.76" rot="R90"/>
 <instance part="LED1" gate="U1" x="220.98" y="137.16" rot="MR0"/>
@@
 <attribute name="VALUE" x="246.38" y="149.86" size="1.778" layer="96" rot="R180"/>
 </instance>
-<instance part="GND2" gate="1" x="231.14" y="104.14"/>
+<instance part="GND2" gate="1" x="231.14" y="101.6"/>
 <instance part="P+5" gate="1" x="231.14" y="116.84" smashed="yes">
 <attribute name="VALUE" x="233.68" y="119.38" size="1.778" layer="96" rot="R180"/>
@@
 </instance>
 <instance part="GND3" gate="1" x="241.3" y="160.02"/>
-<instance part="TP1" gate="G$1" x="254" y="106.68" rot="R90"/>
-<instance part="TP2" gate="G$1" x="254" y="109.22" rot="R90"/>
-<instance part="TP3" gate="G$1" x="254" y="111.76" rot="R90"/>
+<instance part="GND" gate="G$1" x="254" y="104.14" rot="R90"/>
+<instance part="+5V" gate="G$1" x="254" y="109.22" rot="R90"/>
+<instance part="DAT" gate="G$1" x="254" y="114.3" rot="R90"/>
+<instance part="IN" gate="G$1" x="228.6" y="71.12" rot="R90"/>
 </instances>
 <busses>
@@
 <segment>
 <pinref part="GND2" gate="1" pin="GND"/>
-<wire x1="231.14" y1="106.68" x2="251.46" y2="106.68" width="0.1524" layer="91"/>
-<label x="233.68" y="106.68" size="1.778" layer="95"/>
-<pinref part="TP1" gate="G$1" pin="TP"/>
+<wire x1="231.14" y1="104.14" x2="251.46" y2="104.14" width="0.1524" layer="91"/>
+<label x="233.68" y="104.14" size="1.778" layer="95"/>
+<pinref part="GND" gate="G$1" pin="TP"/>
 </segment>
 <segment>
@@
 <wire x1="231.14" y1="109.22" x2="231.14" y2="114.3" width="0.1524" layer="91"/>
 <label x="233.68" y="109.22" size="1.778" layer="95"/>
-<pinref part="TP2" gate="G$1" pin="TP"/>
+<pinref part="+5V" gate="G$1" pin="TP"/>
 </segment>
 <segment>
@@
 <net name="VUSB3V3" class="0">
 <segment>
-<wire x1="193.04" y1="99.06" x2="208.28" y2="99.06" width="0.1524" layer="91"/>
-<wire x1="208.28" y1="99.06" x2="208.28" y2="96.52" width="0.1524" layer="91"/>
+<wire x1="193.04" y1="99.06" x2="220.98" y2="99.06" width="0.1524" layer="91"/>
+<wire x1="220.98" y1="99.06" x2="220.98" y2="96.52" width="0.1524" layer="91"/>
 <pinref part="U1" gate="G$1" pin="VUSB3V3"/>
 <pinref part="C3" gate="G$1" pin="1"/>
+<label x="210.82" y="99.06" size="1.778" layer="95"/>
 </segment>
 </net>
@@
 <wire x1="193.04" y1="93.98" x2="200.66" y2="93.98" width="0.1524" layer="91"/>
 <label x="195.58" y="93.98" size="1.778" layer="95"/>
+<pinref part="IN" gate="G$1" pin="TP"/>
+<wire x1="226.06" y1="71.12" x2="215.9" y2="71.12" width="0.1524" layer="91"/>
+<wire x1="215.9" y1="71.12" x2="215.9" y2="93.98" width="0.1524" layer="91"/>
+<wire x1="215.9" y1="93.98" x2="200.66" y2="93.98" width="0.1524" layer="91"/>
 </segment>
 </net>
 <net name="DO" class="0">
 <segment>
-<label x="233.68" y="111.76" size="1.778" layer="95"/>
-<wire x1="251.46" y1="111.76" x2="233.68" y2="111.76" width="0.1524" layer="91"/>
-<pinref part="TP3" gate="G$1" pin="TP"/>
+<label x="233.68" y="114.3" size="1.778" layer="95"/>
+<wire x1="251.46" y1="114.3" x2="233.68" y2="114.3" width="0.1524" layer="91"/>
+<pinref part="DAT" gate="G$1" pin="TP"/>
 </segment>
 <segment>
@@
 </segment>
 </net>
+<net name="N$2" class="0">
+<segment>
+<pinref part="U1" gate="G$1" pin="RA5"/>
+<wire x1="137.16" y1="104.14" x2="129.54" y2="104.14" width="0.1524" layer="91"/>
+</segment>
+</net>
+<net name="N$3" class="0">
+<segment>
+<pinref part="U1" gate="G$1" pin="RC3"/>
+<wire x1="137.16" y1="91.44" x2="129.54" y2="91.44" width="0.1524" layer="91"/>
+</segment>
+</net>
+<net name="N$6" class="0">
+<segment>
+<pinref part="U1" gate="G$1" pin="RC5"/>
+<wire x1="137.16" y1="96.52" x2="129.54" y2="96.52" width="0.1524" layer="91"/>
+</segment>
+</net>
+<net name="N$4" class="0">
+<segment>
+<pinref part="U1" gate="G$1" pin="RC4"/>
+<wire x1="137.16" y1="93.98" x2="129.54" y2="93.98" width="0.1524" layer="91"/>
+</segment>
+</net>
+<net name="N$5" class="0">
+<segment>
+<pinref part="U1" gate="G$1" pin="RA4"/>
+<wire x1="137.16" y1="101.6" x2="129.54" y2="101.6" width="0.1524" layer="91"/>
+</segment>
+</net>
