File: hardware/schematic/blink1_v2c3.sch (EAGLE design)
At the start: 10 parts, among them P1 TPTP11SQ, U1 PIC16F1455ML, X1 USB

Commit message: misc updates to schems
Parts:
- JP1: value (none) -> strip
Changed lines of the file:
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@@
 <part name="P+7" library="supply1" deviceset="+5V" device=""/>
 <part name="GND3" library="SparkFun-20110517" deviceset="GND" device=""/>
-<part name="JP1" library="SparkFun-20110517" deviceset="M03" device="PTH"/>
+<part name="JP1" library="SparkFun-20110517" deviceset="M03" device="PTH" value="strip"/>
 </parts>
 <sheets>
