File: hardware/schematic/blink1mk2_v2c4.brd (EAGLE design)
At the start: 12.6 x 13.7 mm, 10 parts, among them P1 TPTP11SQ, U1 PIC16F1455ML, X1 USB

Commit message: schematic syncup
Changed lines of the file:
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@@
 <setting verticaltext="up"/>
 </settings>
-<grid distance="0.05" unitdist="inch" unit="inch" style="lines" multiple="10" display="yes" altdistance="0.01" altunitdist="inch" altunit="inch"/>
+<grid distance="0.05" unitdist="inch" unit="mm" style="lines" multiple="10" display="yes" altdistance="0.01" altunitdist="inch" altunit="inch"/>
 <layers>
 <layer number="1" name="Top" color="4" fill="1" visible="yes" active="yes"/>
@@
 <layer number="46" name="Milling" color="3" fill="1" visible="no" active="yes"/>
 <layer number="47" name="Measures" color="7" fill="1" visible="yes" active="yes"/>
-<layer number="48" name="Document" color="7" fill="1" visible="yes" active="yes"/>
+<layer number="48" name="Document" color="7" fill="1" visible="no" active="yes"/>
 <layer number="49" name="Reference" color="7" fill="1" visible="yes" active="yes"/>
 <layer number="50" name="dxf" color="7" fill="1" visible="no" active="yes"/>
@@
 <layer number="155" name="FabDoc3" color="7" fill="1" visible="no" active="yes"/>
 <layer number="199" name="Contour" color="7" fill="1" visible="no" active="yes"/>
-<layer number="200" name="200bmp" color="6" fill="10" visible="no" active="yes"/>
+<layer number="200" name="200bmp" color="6" fill="10" visible="yes" active="yes"/>
 <layer number="201" name="201bmp" color="2" fill="1" visible="no" active="no"/>
 <layer number="202" name="202bmp" color="3" fill="1" visible="no" active="no"/>
-<layer number="203" name="203bmp" color="4" fill="10" visible="no" active="yes"/>
-<layer number="204" name="204bmp" color="5" fill="10" visible="no" active="yes"/>
-<layer number="205" name="205bmp" color="6" fill="10" visible="no" active="yes"/>
-<layer number="206" name="206bmp" color="7" fill="10" visible="no" active="yes"/>
+<layer number="203" name="203bmp" color="4" fill="10" visible="yes" active="yes"/>
+<layer number="204" name="204bmp" color="5" fill="10" visible="yes" active="yes"/>
+<layer number="205" name="205bmp" color="6" fill="10" visible="yes" active="yes"/>
+<layer number="206" name="206bmp" color="7" fill="10" visible="yes" active="yes"/>
 <layer number="207" name="207bmp" color="8" fill="10" visible="yes" active="yes"/>
 <layer number="208" name="208bmp" color="9" fill="10" visible="yes" active="yes"/>
@@
 <plain>
 <text x="6.9596" y="3.5661" size="0.6096" layer="21" ratio="10" rot="SR90">blink1.thingm.com</text>
-<text x="7.874" y="11.176" size="0.889" layer="21" ratio="10">blink(1)</text>
-<text x="1.524" y="3.556" size="0.6096" layer="22" ratio="10" rot="MR90">blink1mk2_v2c4</text>
+<text x="7.62" y="11.176" size="0.889" layer="21" ratio="10">blink(1)</text>
+<text x="1.524" y="3.81" size="0.6096" layer="22" ratio="10" rot="MR90">blink1mk2_v2c4</text>
 <rectangle x1="7.5787" y1="12.3031" x2="9.4837" y2="12.3095" layer="200"/>
 <rectangle x1="7.5787" y1="12.3095" x2="9.4837" y2="12.3158" layer="200"/>
@@
 <dimension x1="13.208" y1="0.762" x2="13.208" y2="14.478" x3="16.51" y3="7.62" textsize="0.6096" layer="51" dtype="vertical" width="0.0762" unit="inch" visible="yes"/>
 <dimension x1="1.143" y1="13.208" x2="13.716" y2="12.7" x3="7.4295" y3="15.748" textsize="0.6096" layer="51" dtype="horizontal" width="0.0762" unit="inch" visible="yes"/>
-<polygon width="0.254" layer="51">
+<polygon width="0.254" layer="48">
 <vertex x="12.192" y="3.048"/>
 <vertex x="14.732" y="3.048"/>
@@
 <vertex x="12.192" y="0.508"/>
 </polygon>
-<polygon width="0.254" layer="51">
+<polygon width="0.254" layer="48">
 <vertex x="12.192" y="14.732"/>
 <vertex x="12.192" y="12.446"/>
@@
 <vertex x="14.732" y="14.732"/>
 </polygon>
-<dimension x1="13.716" y1="1.778" x2="11.938" y2="1.27" x3="12.827" y3="-1.27" textsize="1.016" layer="51" dtype="horizontal" width="0.0508" unit="inch" visible="yes"/>
+<dimension x1="13.716" y1="1.778" x2="11.938" y2="1.27" x3="12.827" y3="-1.27" textsize="0.6096" layer="48" dtype="horizontal" width="0.0508" unit="inch" visible="yes"/>
 </plain>
 <attributes>
@@
 </element>
 <element name="JP1" library="todstuff" package="1X03-1.27MM" value="M03" x="8.382" y="2.032" smashed="yes">
-<attribute name="NAME" x="7.874" y="-0.254" size="0.4064" layer="25"/>
 <attribute name="VALUE" x="7.874" y="0.381" size="0.4064" layer="27"/>
 </element>
@@
 <wire x1="7.284" y1="7.295" x2="8.636" y2="7.295" width="0.254" layer="16"/>
 <wire x1="8.636" y1="7.295" x2="8.636" y2="7.366" width="0.254" layer="16"/>
-<wire x1="6.604" y1="12.7" x2="6.604" y2="13.462" width="0.254" layer="1"/>
-<wire x1="6.604" y1="13.462" x2="5.588" y2="13.462" width="0.254" layer="1"/>
+<wire x1="6.858" y1="13.462" x2="5.588" y2="13.462" width="0.254" layer="1"/>
 <wire x1="7.112" y1="11.938" x2="7.112" y2="12.7" width="0.254" layer="1"/>
-<wire x1="7.112" y1="12.7" x2="6.604" y2="12.7" width="0.254" layer="1"/>
+<wire x1="7.112" y1="12.7" x2="7.112" y2="13.208" width="0.254" layer="1"/>
 <wire x1="5.754" y1="12.358" x2="6.096" y2="12.7" width="0.254" layer="16"/>
 <wire x1="6.096" y1="12.7" x2="6.604" y2="12.7" width="0.254" layer="16"/>
@@
 <wire x1="7.112" y1="8.128" x2="7.112" y2="8.636" width="0.254" layer="1"/>
 <wire x1="5.754" y1="12.358" x2="5.754" y2="11.684" width="0.254" layer="16"/>
+<wire x1="6.858" y1="13.462" x2="7.112" y2="13.208" width="0.254" layer="1"/>
+<wire x1="6.604" y1="12.7" x2="7.112" y2="12.7" width="0.254" layer="1"/>
 </signal>
 <signal name="VUSB3V3">
