File: hardware/schematic/blink1mk2_v2c5.brd (EAGLE design)
At the start: 12.6 x 13.7 mm, 10 parts, among them P1 TPTP11SQ, U1 PIC16F1455ML, X1 USB

Commit message: schematic syncup
Parts:
- moved C1 0.25 mm to (11.2, 12.7)
- moved C2 0.25 mm to (9.14, 12.7)
